Commit message: Setup moveit

File: hydra_description/urdf/hydra_description.urdf (robot description, URDF)
Before this commit: robot hydra_description, 9 links, 8 joints
Joints:
- joint joint_0: limit lower=-1.57 upper=1.57 effort=0 velocity=0 -> lower=-1.57 upper=1.57 effort=${effort} velocity=${velocity}
- joint joint_1: limit lower=-1.57 upper=1.57 effort=0 velocity=0 -> lower=-1.57 upper=1.57 effort=${effort} velocity=${velocity}; origin xyz=0 -0.05 0 rpy=1.8356 0 3.1416 -> xyz=-0.02 -0.05 0 rpy=1.8356 0 3.1416
- joint joint_2: limit lower=-1.57 upper=1.57 effort=0 velocity=0 -> lower=-1.57 upper=1.57 effort=${effort} velocity=${velocity}; origin xyz=0 0.0063552 -0.18258 rpy=-0.5902 0 3.1416 -> xyz=-0.02 0.0063552 -0.18258 rpy=-0.5902 0 3.1416
- joint joint_3: limit lower=-1.57 upper=1.57 effort=0 velocity=0 -> lower=-1.57 upper=1.57 effort=${effort} velocity=${velocity}
- joint joint_4: limit lower=-1.57 upper=1.57 effort=0 velocity=0 -> lower=-1.57 upper=1.57 effort=${effort} velocity=${velocity}
- joint joint_5: limit lower=-1.57 upper=1.57 effort=0 velocity=0 -> lower=-1.57 upper=1.57 effort=${effort} velocity=${velocity}
- joint joint_6: limit lower=-1.57 upper=1.57 effort=0 velocity=0 -> lower=-1.57 upper=1.57 effort=${effort} velocity=${velocity}
